Commit message: W2: 车模型改用 TB3 waffle 基座；补 ADR-0011/0012
- agc_car 以 ROS 官方 nav2_minimal_tb3_sim 的 TB3 waffle 为结构基座（轮/关节位姿、
  接触摩擦、DiffDrive 限幅沿用），改名 car/*；mass 取旧树事实 2.0；保留 3D 激光定义；
  参数同步（wheel_separation 0.287 / wheel_radius 0.033 / spawn z 0.010）。
- ADR-0011：显式锁定节点语言（C++ 实时域 / Python RL 域），补足 W0 §9 的口径。
- ADR-0012：PX4 本体以 toolchain 外部依赖形态纳入（pin v1.15.4），px4_msgs 内联 src/。
- 契约 #decisions、Runbook W3、W2 spec R2 同步引用。

File: src/agc_sim/models/agc_car/agc_car.sdf.xacro (robot description, xacro)
@@ -1,67 +1,69 @@
 <?xml version="1.0"?>
 <!--
-  agc_car —— 地面车模型（真实物理，ADR-0010；W2-min）
-  实现说明（全新重写，HOW 不继承旧树）：
-    * 差速两驱动轮 + 前后 2 caster；挂 gz-sim DiffDrive 插件，由物理引擎产生运动。
-    * 参数全部经 xacro 注入，默认值来自 agc_sim/config/car.yaml，由 launch 单一设置。
-    * link 命名遵循契约：机体系为 car/base_link（禁止裸 base_link）。
-    * base_link 原点取轮轴高度；spawn z = wheel_radius 使车轮触地。
-    * 几何/质量沿用旧树 agc_car 的碰撞盒口径（0.44×0.34×0.16、mass 2.0）作为行为事实；
-      visual 改用基本几何（网格细化属 W2-full，不复制旧资产）。
+  agc_car —— 地面车模型（真实物理，ADR-0010；W2）
+  基座来源：以 ROS 官方 `nav2_minimal_tb3_sim` 的 `urdf/gz_waffle.sdf.xacro`
+  （TurtleBot3 waffle，Apache-2.0）为**结构基座**——沿用其差速两驱动轮 + 2 后万向球
+  的布局、轮/关节位姿、接触与摩擦参数、DiffDrive 限幅；**不再从零手搓几何**。
+  相对基座的改动：
+    * 命名改为契约要求：模型 `agc_car`，机体系 `car/base_link`（禁止裸 base_link）；
+    * 车体质量取旧树行为事实 2.0（TB3 原为 1.0）；碰撞盒沿用车体尺寸（0.265×0.265×0.089）；
+    * 传感器：改用 3D 激光（Velodyne 语义，`gpu_lidar`）→ PointCloud2，挂 `car/lidar_link`
+      （TB3 原为 2D `LaserScan` + depth 相机，此处不采用）；
+    * visual 暂用基本几何（TB3 的 dae 网格为 `package://`，gz 不解析；网格细化延后）。
+    * 不设 DiffDrive 的 topic/frame 覆盖，沿用默认 `/model/agc_car/{cmd_vel,odometry}`
+      与 `_publisher` 默认帧（与 agc_sim 桥一致）。
 -->
 <sdf version="1.8" xmlns:xacro="http://www.ros.org/wiki/xacro">
-  <xacro:arg name="wheel_separation" default="0.32"/>
-  <xacro:arg name="wheel_radius" default="0.05"/>
-  <xacro:arg name="wheel_width" default="0.03"/>
+  <xacro:arg name="wheel_separation" default="0.287"/>
+  <xacro:arg name="wheel_radius" default="0.033"/>
+  <xacro:arg name="wheel_width" default="0.018"/>
   <xacro:arg name="max_wheel_torque" default="20.0"/>
   <xacro:arg name="max_wheel_acceleration" default="1.0"/>
-  <xacro:arg name="body_length" default="0.44"/>
-  <xacro:arg name="body_width" default="0.34"/>
-  <xacro:arg name="body_height" default="0.16"/>
+  <xacro:arg name="body_length" default="0.265"/>
+  <xacro:arg name="body_width" default="0.265"/>
+  <xacro:arg name="body_height" default="0.089"/>
   <xacro:arg name="body_mass" default="2.0"/>
   <model name="agc_car">
     <static>false</static>
-    <!-- 车体（原点在轮轴高度） -->
+    <!-- 车体（基座：TB3 base_link；原点约在轮轴高度） -->
     <link name="car/base_link">
       <inertial>
+        <pose>0 0 0.048 0 0 0</pose>
+        <inertia>
+          <ixx>0.001</ixx><ixy>0.0</ixy><ixz>0.0</ixz>
+          <iyy>0.001</iyy><iyz>0.0</iyz><izz>0.001</izz>
+        </inertia>
         <mass>$(arg body_mass)</mass>
-        <inertia>
-          <ixx>0.025</ixx>
-          <iyy>0.025</iyy>
-          <izz>0.04</izz>
-        </inertia>
       </inertial>
-      <collision name="body_collision">
-        <pose>0 0 0.05 0 0 0</pose>
+      <collision name="base_collision">
+        <pose>0 0 0.048 0 0 0</pose>
         <geometry>
           <box><size>$(arg body_length) $(arg body_width) $(arg body_height)</size></box>
         </geometry>
       </collision>
-      <visual name="body_visual">
-        <pose>0 0 0.05 0 0 0</pose>
+      <visual name="base_visual">
+        <pose>0 0 0.048 0 0 0</pose>
         <geometry>
           <box><size>$(arg body_length) $(arg body_width) $(arg body_height)</size></box>
         </geometry>
-        <material>
-          <ambient>0.2 0.2 0.2 1</ambient>
-          <diffuse>0.3 0.3 0.3 1</diffuse>
-        </material>
+        <material><ambient>0.3 0.3 0.3 1</ambient><diffuse>0.4 0.4 0.4 1</diffuse></material>
       </visual>
     </link>
-    <!-- 左驱动轮（link 不旋转；仅几何旋 90° 使圆柱轴沿 y，关节轴才正确） -->
+    <!-- 左驱动轮（基座：wheel_left_link；位姿由 joint pose 给定，link 不重复给 pose） -->
     <link name="car/left_wheel">
-      <pose>0 0.16 0 0 0 0</pose>
       <inertial>
-        <mass>0.2</mass>
-        <inertia><ixx>0.0003</ixx><iyy>0.0003</iyy><izz>0.0003</izz></inertia>
+        <pose>0 0 0 0 0 0</pose>
+        <inertia><ixx>0.001</ixx><iyy>0.001</iyy><izz>0.001</izz></inertia>
+        <mass>0.1</mass>
       </inertial>
-      <collision name="collision">
+      <collision name="wheel_left_collision">
         <pose>0 0 0 1.5708 0 0</pose>
         <geometry><cylinder><radius>$(arg wheel_radius)</radius><length>$(arg wheel_width)</length></cylinder></geometry>
         <surface>
-          <friction><ode><mu>1.0</mu><mu2>1.0</mu2></ode></friction>
+          <friction><ode><mu>1</mu><mu2>1</mu2><slip1>0.035</slip1><slip2>0</slip2><fdir1>0 0 1</fdir1></ode></friction>
+          <contact><ode><soft_cfm>0</soft_cfm><soft_erp>0.2</soft_erp><kp>1e+5</kp><kd>1</kd><max_vel>0.01</max_vel><min_depth>0.001</min_depth></ode></contact>
         </surface>
       </collision>
-      <visual name="visual">
+      <visual name="wheel_left_visual">
         <pose>0 0 0 1.5708 0 0</pose>
         <geometry><cylinder><radius>$(arg wheel_radius)</radius><length>$(arg wheel_width)</length></cylinder></geometry>
@@ -71,17 +73,18 @@
     <!-- 右驱动轮 -->
     <link name="car/right_wheel">
-      <pose>0 -0.16 0 0 0 0</pose>
       <inertial>
-        <mass>0.2</mass>
-        <inertia><ixx>0.0003</ixx><iyy>0.0003</iyy><izz>0.0003</izz></inertia>
+        <pose>0 0 0 0 0 0</pose>
+        <inertia><ixx>0.001</ixx><iyy>0.001</iyy><izz>0.001</izz></inertia>
+        <mass>0.1</mass>
       </inertial>
-      <collision name="collision">
+      <collision name="wheel_right_collision">
         <pose>0 0 0 1.5708 0 0</pose>
         <geometry><cylinder><radius>$(arg wheel_radius)</radius><length>$(arg wheel_width)</length></cylinder></geometry>
         <surface>
-          <friction><ode><mu>1.0</mu><mu2>1.0</mu2></ode></friction>
+          <friction><ode><mu>1</mu><mu2>1</mu2><slip1>0.035</slip1><slip2>0</slip2><fdir1>0 0 1</fdir1></ode></friction>
+          <contact><ode><soft_cfm>0</soft_cfm><soft_erp>0.2</soft_erp><kp>1e+5</kp><kd>1</kd><max_vel>0.01</max_vel><min_depth>0.001</min_depth></ode></contact>
         </surface>
       </collision>
-      <visual name="visual">
+      <visual name="wheel_right_visual">
         <pose>0 0 0 1.5708 0 0</pose>
         <geometry><cylinder><radius>$(arg wheel_radius)</radius><length>$(arg wheel_width)</length></cylinder></geometry>
@@ -89,66 +92,30 @@
       </visual>
     </link>
-    <!-- 前 caster（被动支撑） -->
-    <link name="car/front_caster">
-      <pose>0.18 0 -0.03 0 0 0</pose>
+    <!-- 后万向球（被动支撑；基座：caster_back_*） -->
+    <link name="car/caster_back_left">
+      <pose>0.177 0.064 -0.004 0 0 0</pose>
       <inertial>
-        <mass>0.05</mass>
+        <mass>0.001</mass>
         <inertia><ixx>1e-5</ixx><iyy>1e-5</iyy><izz>1e-5</izz></inertia>
       </inertial>
       <collision name="collision">
-        <geometry><sphere><radius>0.02</radius></sphere></geometry>
-        <surface><friction><ode><mu>0.0</mu><mu2>0.0</mu2></ode></friction></surface>
+        <geometry><sphere><radius>0.005</radius></sphere></geometry>
+        <surface><contact><ode><soft_cfm>0</soft_cfm><soft_erp>0.2</soft_erp><kp>1e+5</kp><kd>1</kd><max_vel>0.01</max_vel><min_depth>0.001</min_depth></ode></contact></surface>
       </collision>
-      <visual name="visual">
-        <geometry><sphere><radius>0.02</radius></sphere></geometry>
-        <material><ambient>0.3 0.3 0.3 1</ambient><diffuse>0.3 0.3 0.3 1</diffuse></material>
-      </visual>
     </link>
-    <!-- 后 caster（被动支撑） -->
-    <link name="car/rear_caster">
-      <pose>-0.18 0 -0.03 0 0 0</pose>
+    <link name="car/caster_back_right">
+      <pose>0.177 -0.064 -0.004 0 0 0</pose>
       <inertial>
-        <mass>0.05</mass>
+        <mass>0.001</mass>
         <inertia><ixx>1e-5</ixx><iyy>1e-5</iyy><izz>1e-5</izz></inertia>
       </inertial>
       <collision name="collision">
-        <geometry><sphere><radius>0.02</radius></sphere></geometry>
-        <surface><friction><ode><mu>0.0</mu><mu2>0.0</mu2></ode></friction></surface>
+        <geometry><sphere><radius>0.005</radius></sphere></geometry>
+        <surface><contact><ode><soft_cfm>0</soft_cfm><soft_erp>0.2</soft_erp><kp>1e+5</kp><kd>1</kd><max_vel>0.01</max_vel><min_depth>0.001</min_depth></ode></contact></surface>
       </collision>
-      <visual name="visual">
-        <geometry><sphere><radius>0.02</radius></sphere></geometry>
-        <material><ambient>0.3 0.3 0.3 1</ambient><diffuse>0.3 0.3 0.3 1</diffuse></material>
-      </visual>
     </link>
-    <!-- 关节（显式 pose 使关节帧 = 轮心，轴沿 y） -->
-    <joint name="left_wheel_joint" type="revolute">
-      <pose>0 0.16 0 0 0 0</pose>
-      <parent>car/base_link</parent>
-      <child>car/left_wheel</child>
-      <axis>
-        <xyz>0 1 0</xyz>
-        <limit><lower>-1e16</lower><upper>1e16</upper></limit>
-      </axis>
-    </joint>
-    <joint name="right_wheel_joint" type="revolute">
-      <pose>0 -0.16 0 0 0 0</pose>
-      <parent>car/base_link</parent>
-      <child>car/right_wheel</child>
-      <axis>
-        <xyz>0 1 0</xyz>
-        <limit><lower>-1e16</lower><upper>1e16</upper></limit>
-      </axis>
-    </joint>
-    <joint name="front_caster_joint" type="fixed">
-      <parent>car/base_link</parent>
-      <child>car/front_caster</child>
-    </joint>
-    <joint name="rear_caster_joint" type="fixed">
-      <parent>car/base_link</parent>
-      <child>car/rear_caster</child>
-    </joint>
-    <!-- 3D 激光（Velodyne 语义；W2-full 传感器链路）——挂车体，供 W4 costmap / W5 collision_monitor -->
+    <!-- 3D 激光（W2-full 传感器链路；供 W4 costmap / W5 collision_monitor） -->
     <link name="car/lidar_link">
-      <pose>0 0 0.20 0 0 0</pose>
+      <pose>0 0 0.12 0 0 0</pose>
       <inertial>
         <mass>0.1</mass>
@@ -162,14 +129,6 @@
         <lidar>
           <scan>
-            <horizontal>
-              <samples>360</samples>
-              <min_angle>-3.14159265</min_angle>
-              <max_angle>3.14159265</max_angle>
-            </horizontal>
-            <vertical>
-              <samples>16</samples>
-              <min_angle>-0.261799</min_angle>
-              <max_angle>0.261799</max_angle>
-            </vertical>
+            <horizontal><samples>360</samples><min_angle>-3.14159265</min_angle><max_angle>3.14159265</max_angle></horizontal>
+            <vertical><samples>16</samples><min_angle>-0.261799</min_angle><max_angle>0.261799</max_angle></vertical>
           </scan>
           <range><min>0.2</min><max>20.0</max></range>
@@ -177,9 +136,30 @@
       </sensor>
     </link>
+    <!-- 关节（基座布局；轮用 revolute，顺时针/逆时针由 DiffDrive 驱动） -->
+    <joint name="left_wheel_joint" type="revolute">
+      <pose>0 0.144 0.023 0 0 0</pose>
+      <parent>car/base_link</parent>
+      <child>car/left_wheel</child>
+      <axis><xyz>0 1 0</xyz><limit><lower>-1e16</lower><upper>1e16</upper></limit></axis>
+    </joint>
+    <joint name="right_wheel_joint" type="revolute">
+      <pose>0 -0.144 0.023 0 0 0</pose>
+      <parent>car/base_link</parent>
+      <child>car/right_wheel</child>
+      <axis><xyz>0 1 0</xyz><limit><lower>-1e16</lower><upper>1e16</upper></limit></axis>
+    </joint>
+    <joint name="caster_back_left_joint" type="ball">
+      <parent>car/base_link</parent>
+      <child>car/caster_back_left</child>
+    </joint>
+    <joint name="caster_back_right_joint" type="ball">
+      <parent>car/base_link</parent>
+      <child>car/caster_back_right</child>
+    </joint>
     <joint name="lidar_joint" type="fixed">
       <parent>car/base_link</parent>
       <child>car/lidar_link</child>
     </joint>
-    <!-- 差速驱动插件（真实物理） -->
+    <!-- 差速驱动（真实物理；限幅沿用 TB3 基座量级） -->
     <plugin filename="gz-sim-diff-drive-system" name="gz::sim::systems::DiffDrive">
       <left_joint>left_wheel_joint</left_joint>
@@ -189,12 +169,9 @@
       <max_wheel_torque>$(arg max_wheel_torque)</max_wheel_torque>
       <max_wheel_acceleration>$(arg max_wheel_acceleration)</max_wheel_acceleration>
+      <max_linear_velocity>0.5</max_linear_velocity>
+      <min_linear_velocity>-0.5</min_linear_velocity>
+      <max_angular_velocity>2.0</max_angular_velocity>
+      <min_angular_velocity>-2.0</min_angular_velocity>
       <odom_publish_frequency>30</odom_publish_frequency>
-    </plugin>
-    <!-- 世界真值位姿发布（供 M0 的 ground_odom_adapter 取 world 位姿；teleport 安全）。
-         update_frequency 使位姿按固定频率发布（否则仅在位姿变化时发布，静止车无输出）。 -->
-    <plugin filename="gz-sim-pose-publisher-system" name="gz::sim::systems::PosePublisher">
-      <publish_model_pose>true</publish_model_pose>
-      <publish_link_pose>false</publish_link_pose>
-      <update_frequency>30</update_frequency>
     </plugin>
   </model>

Commit message: W2-interception: intruder_uav 可控化 + 地面平台拦截载荷模型
- intruder_uav 挂 GZ VelocityControl（gz /model/intruder_uav/cmd_vel ↔ ROS /agc/sim/target_cmd_vel），
  目标可脚本化驱动（driver / 干扰注入节点属 W6）。
- agc_car 增 car/capture_net（直径 2m 圆面，法线 +x）与 car/jammer（轻量、无碰撞）；
  参数 capture_net_radius/payload_mass 落 config/car.yaml 并由 launch 单一设置。
- spec 新增 R9/R10 与 W2-interception 分段；tasks/checklist/GLOSSARY/README/Runbook 同步。
- 一并纳入 ADR-0013..0017 与相关契约/术语/Runbook/AGENTS 改动（本次研究后新决定）。

实测：目标 Twist 驱动位姿 (6.5,2.5)->(13.18,2.5)；两载荷 link 就位；点云 10Hz；车仍受驱运动（未破坏 R2）。

File: src/agc_sim/models/agc_car/agc_car.sdf.xacro (robot description, xacro)
@@ -24,7 +24,10 @@
   <xacro:arg name="body_height" default="0.089"/>
   <xacro:arg name="body_mass" default="2.0"/>
+  <!-- 拦截载荷（W2-interception，R10）：轻量附件、无碰撞；参数落 config -->
+  <xacro:arg name="capture_net_radius" default="1.0"/>
+  <xacro:arg name="payload_mass" default="0.05"/>
   <model name="agc_car">
     <static>false</static>
-    <!-- 车体（基座：TB3 base_link；原点约在轮轴高度） -->
+    <!-- 车体（基座：TB3 车身 link；原点约在轮轴高度） -->
     <link name="car/base_link">
       <inertial>
@@ -136,4 +139,30 @@
       </sensor>
     </link>
+    <!-- 拦截载荷（W2-interception，R10）：轻量附件、**无碰撞**、不改动 DiffDrive 标定 -->
+    <!-- 捕获网面：直径 2 m 的圆面，法线朝前（+x），供 W6 物理捕获"穿越判据"使用 -->
+    <link name="car/capture_net">
+      <pose>0.45 0 0.10 0 0 0</pose>
+      <inertial>
+        <mass>$(arg payload_mass)</mass>
+        <inertia><ixx>1e-4</ixx><iyy>1e-4</iyy><izz>1e-4</izz></inertia>
+      </inertial>
+      <visual name="capture_net_visual">
+        <pose>0 0 0 0 1.5708 0</pose>
+        <geometry><cylinder><radius>$(arg capture_net_radius)</radius><length>0.01</length></cylinder></geometry>
+        <material><ambient>0.1 0.5 0.9 0.5</ambient><diffuse>0.1 0.5 0.9 0.5</diffuse></material>
+      </visual>
+    </link>
+    <!-- 干扰载荷：行为级电子干扰发射器（EMI 不建模）；行为接口属 W6 -->
+    <link name="car/jammer">
+      <pose>-0.10 0 0.16 0 0 0</pose>
+      <inertial>
+        <mass>$(arg payload_mass)</mass>
+        <inertia><ixx>1e-4</ixx><iyy>1e-4</iyy><izz>1e-4</izz></inertia>
+      </inertial>
+      <visual name="jammer_visual">
+        <geometry><cylinder><radius>0.03</radius><length>0.08</length></cylinder></geometry>
+        <material><ambient>0.8 0.6 0.0 1</ambient><diffuse>0.9 0.7 0.0 1</diffuse></material>
+      </visual>
+    </link>
     <!-- 关节（基座布局；轮用 revolute，顺时针/逆时针由 DiffDrive 驱动） -->
     <joint name="left_wheel_joint" type="revolute">
@@ -160,4 +189,12 @@
       <parent>car/base_link</parent>
       <child>car/lidar_link</child>
+    </joint>
+    <joint name="capture_net_joint" type="fixed">
+      <parent>car/base_link</parent>
+      <child>car/capture_net</child>
+    </joint>
+    <joint name="jammer_joint" type="fixed">
+      <parent>car/base_link</parent>
+      <child>car/jammer</child>
     </joint>
     <!-- 差速驱动（真实物理；限幅沿用 TB3 基座量级） -->

File: src/agc_sim/models/intruder_uav/intruder_uav.sdf.xacro (robot description, xacro)
@@ -1,9 +1,12 @@
 <?xml version="1.0"?>
 <!--
-  intruder_uav —— 阶段 A 真值目标（被动，W2-min）
+  intruder_uav —— 可控目标（W2-interception）
   实现说明（全新重写）：
-    * link 级 <gravity>false</gravity> + 无任何插件：纯被动刚体，保持悬停（SDF 的
-      gravity 属 link 而非 model）。
-    * 位姿由 set_pose 服务搬运（driver 属 W4；复位属 M0）。
+    * link 级 <gravity>false</gravity>：**失重**（SDF 的 gravity 属 link 而非 model）。
+    * **可控化**（R9）：挂 GZ `VelocityControl`，外部经话题 `/model/intruder_uav/cmd_vel`
+      发 Twist 速度指令即可脚本化驱动（半运动学，位置 = 速度积分）。**driver / 干扰注入
+      节点属 W6**（[ADR-0016](../../../docs/adr/0016-execution-scope-exit-w6.md)）；
+      本模型只提供"被控制的能力"。
+    * 位姿亦可用 set_pose 服务直接置位（复位属 M0）。
     * 参数经 xacro 注入（默认值来自 agc_sim/config/target.yaml）。
     * 碰撞盒口径沿用旧树（0.32×0.32×0.10、mass 1.0）作为行为事实；visual 用基本几何+
@@ -42,4 +45,8 @@
       </visual>
     </link>
+    <!-- 可控化（R9）：外部速度指令驱动；driver / 干扰注入节点属 W6（ADR-0016） -->
+    <plugin filename="gz-sim-velocity-control-system" name="gz::sim::systems::VelocityControl">
+      <topic>/model/intruder_uav/cmd_vel</topic>
+    </plugin>
   </model>
 </sdf>
